File: JagLink-SNAC.kicad_pcb (KiCad board)
At the start: 2 copper layers, 54.1 x 33 mm, 13 parts

Commit message: Add GitHub link to silkscreen
Other:
- board text added: "https://github.com/kconger/JagLink-SNAC"
Changed lines of the file:
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@@
 		(layer "Edge.Cuts")
+	)
+	(gr_text "https://github.com/kconger/JagLink-SNAC"
+		(at 172 102.5 0)
+		(layer "B.SilkS")
+		(effects
+			(font
+				(size 1 1)
+				(thickness 0.1875)
+			)
+			(justify left bottom mirror)
+		)
 	)
 	(gr_text "JagLink SNAC for MiSTer"
